File: eliografo.kicad_pcb (KiCad board)
At the start: 2 copper layers, 48.3 x 96.5 mm, 46 parts, among them J10 Conn_01x03, J11 Conn_01x02, J3 Conn_01x05, J4 Conn_01x05, J5 Conn_02x06_Odd_Even, J6 Conn_01x02, J7 Conn_01x02, J8 Conn_01x03, J9 Conn_01x03, Q1 IRF540N, U1 LM2672M-3.3, U2 mini_esp32

Commit message: First sketch of version 0.2
Parts:
- removed C6, C7: 100n, Capacitor_THT:C_Rect_L7.0mm_W2.0mm_P5.00mm
- removed R12: 1k, Resistor_THT:R_Axial_DIN0204_L3.6mm_D1.6mm_P5.08mm_Horizontal
- removed TP1, TP10, TP2, TP6, TP7: TestPoint, TestPoint:TestPoint_THTPad_D2.0mm_Drill1.0mm
- added D2: LED, LED_THT:LED_D3.0mm, F.Cu at (107.6, 87.2)
- added H2: MountingHole_Pad, MountingHole:MountingHole_3.2mm_M3_Pad, F.Cu at (121.2, 92.9)
- added H3: MountingHole_Pad, MountingHole:MountingHole_3.2mm_M3_Pad, F.Cu at (161.2, 52.9)
- added H4: MountingHole_Pad, MountingHole:MountingHole_3.2mm_M3_Pad, F.Cu at (121.2, 52.9)
- added H5: MountingHole_Pad, MountingHole:MountingHole_3.2mm_M3_Pad, F.Cu at (196.0, 53.9)
- added H6: MountingHole_Pad, MountingHole:MountingHole_3.2mm_M3_Pad, F.Cu at (46.0, 53.9)
- added J1: Conn_01x05, Connector_PinSocket_2.54mm:PinSocket_1x05_P2.54mm_Vertical, F.Cu at (75.8, 47.2)
- added J12: EXTRA ADC, Connector_PinHeader_2.54mm:PinHeader_1x02_P2.54mm_Vertical, F.Cu at (89.9, 83.0)
- added J13: Conn_01x03, Connector_PinHeader_2.54mm:PinHeader_1x03_P2.54mm_Vertical, F.Cu at (114.5, 50.1)
- added J2: ADC, Connector_PinSocket_2.54mm:PinSocket_1x10_P2.54mm_Vertical, F.Cu at (79.1, 52.5)
- added JP1: ENC AZI DIRECT, Connector_PinHeader_2.54mm:PinHeader_1x02_P2.54mm_Vertical, F.Cu at (170.6, 79.8)
- added JP2: ENC ALT DIRECT, Connector_PinHeader_2.54mm:PinHeader_1x02_P2.54mm_Vertical, F.Cu at (168.5, 61.8)
- added JP3: BATT DIRECT, Connector_PinHeader_2.54mm:PinHeader_1x02_P2.54mm_Vertical, F.Cu at (61.6, 53.5)
- added JP4: I2C ENABLE, Connector_PinHeader_2.54mm:PinHeader_1x03_P2.54mm_Vertical, F.Cu at (115.7, 100.0)
- added JP5: LED EN, Connector_PinHeader_2.54mm:PinHeader_1x02_P2.54mm_Vertical, F.Cu at (107.8, 83.0)
- added Q2: MMBT3904, Package_TO_SOT_SMD:SOT-23, F.Cu at (147.0, 80.4)
- added Q4: MMBT3904, Package_TO_SOT_SMD:SOT-23, F.Cu at (126.2, 81.2)
- added Q5: IRLML9301, Package_TO_SOT_SMD:SOT-23, F.Cu at (128.9, 85.9)
- C1: value C_Polarized -> 100uF 25V; footprint Capacitor_THT:CP_Radial_D8.0mm_P5.00mm -> Capacitor_Tantalum_SMD:CP_EIA-7361-38_AVX-V_HandSolder
- C2, C8: footprint Capacitor_THT:C_Rect_L7.0mm_W2.0mm_P5.00mm -> Capacitor_SMD:C_0805_2012Metric_Pad1.18x1.45mm_HandSolder
- C3: value C_Polarized -> 100uF 10V; footprint Capacitor_THT:CP_Radial_D8.0mm_P5.00mm -> Capacitor_Tantalum_SMD:CP_EIA-7343-15_Kemet-W_HandSolder
- C4, C5: value 100u -> 100n; footprint Capacitor_THT:CP_Radial_D8.0mm_P5.00mm -> Capacitor_SMD:C_0805_2012Metric_Pad1.18x1.45mm_HandSolder
- D1: value 1N5819 -> SB140; footprint Diode_THT:D_DO-41_SOD81_P10.16mm_Horizontal -> Diode_SMD:D_SMA
- J10: value Conn_01x03 -> Driver PSU; footprint Connector_Phoenix_MSTB:PhoenixContact_MSTBA_2,5_3-G-5,08_1x03_P5.08mm_Horizontal -> TerminalBlock_Phoenix:TerminalBlock_Phoenix_MKDS-1,5-3-5.08_1x03_P5.08mm_Horizontal
- J11: value Conn_01x02 -> POWER SUPPLY; footprint Connector_Phoenix_MSTB:PhoenixContact_MSTBA_2,5_2-G-5,08_1x02_P5.08mm_Horizontal -> TerminalBlock_Phoenix:TerminalBlock_Phoenix_MKDS-1,5-2-5.08_1x02_P5.08mm_Horizontal
- J3, J4: footprint Connector_PinHeader_2.54mm:PinHeader_1x05_P2.54mm_Vertical -> Connector_PinSocket_2.54mm:PinSocket_1x05_P2.54mm_Vertical
- J5: value Conn_02x06_Odd_Even -> MotorDriver; footprint Connector_PinHeader_2.54mm:PinHeader_2x06_P2.54mm_Vertical -> Connector_IDC:IDC-Header_2x06_P2.54mm_Vertical
- J8: value Conn_01x03 -> Encoder ALT; footprint Connector_Phoenix_MSTB:PhoenixContact_MSTBA_2,5_3-G-5,08_1x03_P5.08mm_Horizontal -> TerminalBlock_Phoenix:TerminalBlock_Phoenix_MKDS-1,5-3-5.08_1x03_P5.08mm_Horizontal
- J9: value Conn_01x03 -> Encoder AZI; footprint Connector_Phoenix_MSTB:PhoenixContact_MSTBA_2,5_3-G-5,08_1x03_P5.08mm_Horizontal -> TerminalBlock_Phoenix:TerminalBlock_Phoenix_MKDS-1,5-3-5.08_1x03_P5.08mm_Horizontal
- L1: value INDUCTOR -> 47uH; footprint Inductor_THT:L_Axial_L20.3mm_D12.1mm_P7.62mm_Vertical_Vishay_IHA-101 -> Inductor_SMD:L_Coilcraft_XAL6060-XXX
- Q1: value IRF540N -> IRF9540N; footprint Package_TO_SOT_THT:TO-220-3_Vertical -> Package_TO_SOT_SMD:TO-252-3_TabPin2
- R1, R10, R11, R2, R5, R6, R7, R8: footprint Resistor_THT:R_Axial_DIN0204_L3.6mm_D1.6mm_P5.08mm_Horizontal -> Resistor_SMD:R_0805_2012Metric_Pad1.20x1.40mm_HandSolder
- R3: value 560k -> 330; footprint Resistor_THT:R_Axial_DIN0204_L3.6mm_D1.6mm_P5.08mm_Horizontal -> Resistor_SMD:R_0805_2012Metric_Pad1.20x1.40mm_HandSolder
- R4: value 560k -> 1k; footprint Resistor_THT:R_Axial_DIN0204_L3.6mm_D1.6mm_P5.08mm_Horizontal -> Resistor_SMD:R_0805_2012Metric_Pad1.20x1.40mm_HandSolder
- R9: value 10k -> 1k; footprint Resistor_THT:R_Axial_DIN0204_L3.6mm_D1.6mm_P5.08mm_Horizontal -> Resistor_SMD:R_0805_2012Metric_Pad1.20x1.40mm_HandSolder
- moved J11 119.6 mm to (56.8, 58.9), turned to -90 degrees
- moved J6 107.3 mm to (57.9, 43.6)
- moved J7 102.2 mm to (57.9, 47.2)
- moved C1 97.4 mm to (61.7, 72.4), turned to 180 degrees
- moved L1 88.4 mm to (78.2, 83.2), turned to 0 degrees
- moved U1 87.6 mm to (69.8, 80.5), turned to 180 degrees
- moved J3 87.0 mm to (75.8, 43.7), turned to -90 degrees
- moved D1 81.1 mm to (78.4, 89.1), turned to 0 degrees
- moved C2 80.8 mm to (70.7, 84.5), turned to 180 degrees
- moved R11 78.1 mm to (65.4, 55.1), turned to 0 degrees
- moved J10 75.1 mm to (154.1, 56.6), turned to 180 degrees
- moved C8 73.3 mm to (65.4, 57.4), turned to 180 degrees
- moved R10 73.2 mm to (65.3, 59.7), turned to 180 degrees
- moved R5 72.0 mm to (170.1, 50.2), turned to 180 degrees
- moved TP11 71.2 mm to (192.4, 60.2)
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Connections:
- C4 pad 1: Net-(C4-Pad1) -> ENCODER A
- C5 pad 1: Net-(C5-Pad1) -> ENCODER B
- J10 pad 1: +12V -> +12 DRIVER
- J10 pad 2: Net-(J10-Pin_2) -> GND
- J3 pad 2: +5V -> I2C_3.3
- J4 pad 2: +5V -> I2C_3.3
- Q1 pad 2: Net-(J10-Pin_2) -> +12 DRIVER
- Q1 pad 3: GND -> +12V
- R1 pad 1: Net-(C4-Pad1) -> Net-(Q1-G)
- R1 pad 2: +5V -> +12V
- R2 pad 1: Net-(C5-Pad1) -> Net-(Q4-C)
- R2 pad 2: +5V -> +3.3V
- R3 pad 1: Net-(C4-Pad1) -> GND
- R3 pad 2: ENCODER B -> Net-(D2-K)
- R4 pad 1: Net-(C5-Pad1) -> I2C_3.3_ENABLE
- R4 pad 2: ENCODER A -> Net-(Q4-B)
- R9 pad 2: Net-(Q1-G) -> Net-(Q2-B)
- TP12 pad 1: Net-(J10-Pin_2) -> +12 DRIVER
- U2 pad 10: unconnected-(U2-IO_19/D6-Pad10) -> Net-(JP4-B)
- U2 pad 11: ENCODER A -> Net-(JP1-B)
- U2 pad 21: unconnected-(U2-TXD-Pad21) -> Net-(J13-Pin_1)
- U2 pad 23: unconnected-(U2-RXD-Pad23) -> Net-(J13-Pin_2)
- U2 pad 4: BATTERY LEVEL -> Net-(JP3-B)
- U2 pad 7: ENCODER B -> Net-(JP2-B)
Routing:
- net GND: track 156.3 -> 404.4 mm, vias 1 -> 4
- net I2C_3.3: track 0.00 -> 121.4 mm, vias 0 -> 1
- net Net-(JP2-B): track 0.00 -> 99.4 mm
- net Net-(JP1-B): track 0.00 -> 91.8 mm
- net ENCODER A: track 29.4 -> 113.4 mm
- net ENCODER B: track 60.8 -> 140.0 mm
- net Net-(Q1-G): track 82.0 -> 11.4 mm, vias 1 -> 0
- net Net-(JP4-B): track 0.00 -> 67.7 mm, vias 0 -> 2
- net +12 DRIVER: track 0.00 -> 55.2 mm
- net +5V: track 139.7 -> 85.3 mm
- net +3.3V: track 98.9 -> 145.8 mm, vias 0 -> 2
- net +12V: track 117.3 -> 156.1 mm, vias 0 -> 1
- net SDA: track 76.1 -> 109.9 mm, vias 1 -> 0
- net MOT B D1: track 58.9 -> 31.6 mm, vias 3 -> 0
- net Net-(JP3-B): track 0.00 -> 25.1 mm
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- removed copper zone on B.Cu, net GND
- removed copper zone on F.Cu, net GND
Other:
- board size 48.3 x 96.5 mm -> 168.7 x 62.1 mm
- board text added: "+12V"
- board text added: "+3.3V GND"
- board text added: "+5V"
- board text added: "."
- board text added: "ADS1115 ADC MODULE"
- board text added: "ADS1115 MODULE"
- board text added: "ALT"
- board text added: "ALT ENC -> INTERNAL ADC"
- board text added: "AZI"
- board text added: "AZI ENC -> INTERNAL ADC"
- board text added: "BAT LVL -> INTERNAL ADC"
- board text added: "BOARD POWER"
- board text added: "DAC A03"
- board text added: "DRIVER CONTROL"
- board text added: "DRIVER POWER"
- board text added: "DS1307 RTC MODULE"
- board text added: "ENCODERS"
- board text added: "GND"
- board text added: "GND RXD TXD"
- board text added: "I2C 3.3V"
- board text added: "I2C POWER SUPPLY ENABLE PIN"
- board text added: "IO19"
- board text added: "LED ENABLE"
- board text added: "M. DRIVER (IO4)"
- board text added: "MOTOR ALT"
- board text added: "MOTOR AZI"
- board text added: "RTC"
- board text added: "SERIAL"
- board text added: "SIG"
- board text added: "V+"
- board text added: "X SCL SDA +3.3V GND"

Commit message: Version 0.2 ready for production
Other:
- board text added: "Alessandro Lupi ELIOS"
- board text added: "Designed by Mattia Bondanza 2025 v0.2"
